Commit message: Fix the angle offset of upperarm

File: urdf/arm.urdf (robot description, URDF)
Before this commit: robot ur5, 8 links, 7 joints
Joints:
- joint shoulder_lift_joint: limit lower=-3.14159265 upper=3.14159265 effort=150.0 velocity=3.15 -> lower=${-pi} upper=${pi} effort=150.0 velocity=3.15

Commit message: Update mesh

File: urdf/arm.urdf (robot description, URDF)
Before this commit: robot ur5, 8 links, 7 joints
Links:
- link forearm_link: geometry collision mesh filename=package://enpm662_final_project/mesh/ur5/collision/forearm.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; visual mesh filename=package://enpm662_final_project/mesh/ur5/visual/forearm.dae
- link shoulder_link: geometry collision mesh filename=package://enpm662_final_project/mesh/ur5/collision/shoulder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; visual mesh filename=package://enpm662_final_project/mesh/ur5/visual/shoulder.dae
- link upper_arm_link: geometry collision mesh filename=package://enpm662_final_project/mesh/ur5/collision/upperarm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; visual mesh filename=package://enpm662_final_project/mesh/ur5/visual/upperarm.dae
- link ur5_base_link: geometry collision mesh filename=package://enpm662_final_project/mesh/ur5/collision/base.stl; visual mesh filename=package://enpm662_final_project/mesh/ur5/visual/base.dae
- link wrist_1_link: geometry collision mesh filename=package://enpm662_final_project/mesh/ur5/collision/wrist1.s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; visual mesh filename=package://enpm662_final_project/mesh/ur5/visual/wrist1.dae
- link wrist_2_link: geometry collision mesh filename=package://enpm662_final_project/mesh/ur5/collision/wrist2.s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; visual mesh filename=package://enpm662_final_project/mesh/ur5/visual/wrist2.dae
- link wrist_3_link: geometry collision mesh filename=package://enpm662_final_project/mesh/ur5/collision/wrist3.s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; visual mesh filename=package://enpm662_final_project/mesh/ur5/visual/wrist3.dae
