Commit message: Add ur3 arm

File: test/test_robot.urdf.xacro (robot description, xacro)
@@ -56,4 +56,11 @@
     <child link="rear_left_wheel_link" />
   </joint>
+  <xacro:include filename="$(find ur_description)/urdf/inc/ur3_macro.xacro"/>
+  <xacro:ur3_robot prefix="ur3" />
+    <joint name="armGlue" type="fixed">
+    <parent link="base_link"/>
+    <child link="ur3base_link"/>
+    <origin rpy="0 0 0" xyz="0 0 0.1"/>
+  </joint>
   <gazebo>
     <plugin name="gazebo_ros_control" filename="libgazebo_ros_control.so">

Commit message: Adding controller for arm

File: test/test_robot.urdf.xacro (robot description, xacro)
@@ -1,5 +1,5 @@
 <?xml version="1.0" ?>
 <robot name="mecanum_wheel_robot" xmlns:xacro="http://ros.org/wiki/xacro">
-  <xacro:include filename="$(find fuji_mecanum)/urdf/mecanum_wheel_macro.xacro" />
+  <xacro:include filename="$(find enpm662_final_project)/urdf/mecanum_wheel_macro.xacro" />
   <link name="base_link">
     <visual>
@@ -56,10 +56,9 @@
     <child link="rear_left_wheel_link" />
   </joint>
-  <xacro:include filename="$(find ur_description)/urdf/inc/ur3_macro.xacro"/>
-  <xacro:ur3_robot prefix="ur3" />
+  <xacro:include filename="$(find enpm662_final_project)/urdf/arm.urdf"/>
     <joint name="armGlue" type="fixed">
     <parent link="base_link"/>
-    <child link="ur3base_link"/>
-    <origin rpy="0 0 0" xyz="0 0 0.1"/>
+    <child link="ur5_base_link"/>
+    <origin rpy="0 0 0" xyz="0 0 0.3"/>
   </joint>
   <gazebo>

File: urdf/mecanum_wheel.urdf.xacro (robot description, xacro)
@@ -1,5 +1,5 @@
 <?xml version="1.0" ?>
 <robot name="mecanum_wheel_robot" xmlns:xacro="http://ros.org/wiki/xacro">
-  <xacro:include filename="$(find fuji_mecanum)/urdf/mecanum_wheel_macro.xacro" />
+  <xacro:include filename="$(find enpm662_final_project)/urdf/mecanum_wheel_macro.xacro" />
   <xacro:mecanum_wheel name="front_right" side="1" interface="hardware_interface/EffortJointInterface" />
   <xacro:mecanum_wheel name="front_left" side="-1" interface="hardware_interface/EffortJointInterface" />

File: urdf/mecanum_wheel_macro.xacro (robot description, xacro)
@@ -1,6 +1,6 @@
 <?xml version="1.0" ?>
 <robot name="mecanum_wheel" xmlns:xacro="http://ros.org/wiki/xacro">
-  <xacro:include filename="$(find fuji_mecanum)/urdf/wheel.xacro" />
-  <xacro:include filename="$(find fuji_mecanum)/urdf/rollers.xacro"  />
+  <xacro:include filename="$(find enpm662_final_project)/urdf/wheel.xacro" />
+  <xacro:include filename="$(find enpm662_final_project)/urdf/rollers.xacro"  />
   <xacro:macro name="mecanum_wheel" params="name side interface">
     <xacro:wheel_link name="${name}" side="${side}" />

File: urdf/rollers.xacro (robot description, xacro)
@@ -15,10 +15,10 @@
           <origin xyz="0 0 0" rpy="0 0 0" />
           <geometry>
-            <mesh filename="package://fuji_mecanum/mesh/visual/roller.dae" scale="1 1 1" />
+            <mesh filename="package://enpm662_final_project/mesh/visual/roller.dae" scale="1 1 1" />
           </geometry>
         </visual>
         <collision>
           <geometry>
-            <mesh filename="package://fuji_mecanum/mesh/collision/roller.stl" scale="1 1 1" />
+            <mesh filename="package://enpm662_final_project/mesh/collision/roller.stl" scale="1 1 1" />
           </geometry>
         </collision>

File: urdf/wheel.xacro (robot description, xacro)
@@ -6,10 +6,10 @@
         <origin xyz="0 0 0" rpy="0 0 0" />
         <geometry>
-          <mesh filename="package://fuji_mecanum/mesh/visual/wheel.dae" scale="${side} 1 1" />
+          <mesh filename="package://enpm662_final_project/mesh/visual/wheel.dae" scale="${side} 1 1" />
         </geometry>
       </visual>
       <collision>
         <geometry>
-          <mesh filename="package://fuji_mecanum/mesh/collision/wheel.stl" scale="${side} 1 1" />
+          <mesh filename="package://enpm662_final_project/mesh/collision/wheel.stl" scale="${side} 1 1" />
         </geometry>
       </collision>

Commit message: Clean up workspace

File: test/test_robot.urdf.xacro (robot description, xacro)
@@ -60,5 +60,5 @@
     <parent link="base_link"/>
     <child link="ur5_base_link"/>
-    <origin rpy="0 0 0" xyz="0 0 0.3"/>
+    <origin rpy="0 0 0" xyz="0 0 0.2"/>
   </joint>
   <gazebo>

Commit message: Update README and increase offset for Obj locations

File: test/test_robot.urdf.xacro (robot description, xacro)
@@ -60,5 +60,5 @@
     <parent link="base_link"/>
     <child link="ur5_base_link"/>
-    <origin rpy="0 0 0" xyz="0 0 0.2"/>
+    <origin rpy="0 0 0" xyz="0 0 0.15"/>
   </joint>
   <gazebo>
